File: HE8_bottomplate/HE8_bottomplate.kicad_pcb (KiCad board)
At the start: 2 copper layers, 105.2 x 50 mm, 6 parts

Commit message: add plate arts
Parts:
- added G***: LOGO, LOGO, F.Cu at (160.3, 67.3)
